File: pcb/pcb_for_Polaroid/ShutterCal_Polaroid/ShutterCal_Polaroid.kicad_pcb (KiCad board)
At the start: 2 copper layers, 84.7 x 87 mm, 34 parts, among them J1 Conn_Coaxial, J2 Conn_01x04_Socket, J3 USB_C_Receptacle_USB2.0, J4 Conn_01x04_Socket, J5 Conn_01x04_Socket, J6 Conn_01x04_Shielded, J7 Conn_01x02_Socket, J9 Conn_01x04_Shielded, U1 OPA365xxDBV, U2 STM32G030F6Px, U3 CH340N, U4 AMS1117-3.3

Commit message: Polaroid board: fix R4/R5 reference divider and USB-C CC resistors
- R4/R5: the PCB routes R4 from GND to U1+ and R5 from U1+ to +5V, but
  the schematic had them the other way round (and the PCB footprints
  linked to deleted symbols, so parity matched by reference only). With
  the schematic values as routed, U1+ sat at ~4.9 V and the photodiode
  amp was saturated. The schematic now matches the routed copper: R4
  (6.8k) is on the GND side and R5 (330k) on the +5V side, giving
  ~0.10 V at U1+, which is what the firmware's dark threshold expects.
  The PCB footprints are relinked to the current symbols. Copper is
  unchanged.
- R6/R7 (USB-C CC1/CC2 pull-downs): 1k / not fitted -> 5.1k / 5.1k, as
  the Type-C spec requires for a sink, so C-to-C cables work in both
  plug orientations.

DRC: 0 unconnected, all 4 R4/R5 net conflicts gone; the remaining
warnings are unchanged.

Co-Authored-By: Claude Opus 5.5 <noreply@anthropic.com>
Parts:
- R4: value 330k -> 6.8k
- R5: value 6.8k -> 330k
- R6: value 1k -> 5.1k
- R7: value (1k)DNF -> 5.1k
Changed lines of the file:
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@@
         (effects (font (size 1 1) (thickness 0.15)) (justify mirror))
     )
-    (fp_text value "330k" (at 0 -1.43) (layer "B.Fab")
+    (fp_text value "6.8k" (at 0 -1.43) (layer "B.Fab")
         (effects (font (size 1 1) (thickness 0.15)) (justify mirror))
     )
@@
         (effects (font (size 1 1) (thickness 0.15)) (justify mirror))
     )
-    (fp_text value "1k" (at 0 -1.65 90) (layer "B.Fab")
+    (fp_text value "5.1k" (at 0 -1.65 90) (layer "B.Fab")
         (effects (font (size 1 1) (thickness 0.15)) (justify mirror))
     )
@@
         (effects (font (size 1 1) (thickness 0.15)) (justify mirror))
     )
-    (fp_text value "6.8k" (at 0 -1.43) (layer "B.Fab")
+    (fp_text value "330k" (at 0 -1.43) (layer "B.Fab")
         (effects (font (size 1 1) (thickness 0.15)) (justify mirror))
     )
@@
         (effects (font (size 1 1) (thickness 0.15)) (justify mirror))
     )
-    (fp_text value "(1k)DNF" (at 0 -1.65 90) (layer "B.Fab")
-        (effects (font (size 1 1) (thickness 0.15)) (justify mirror))
-    )
+    (fp_text value "5.1k" (at 0 -1.65 90) (layer "B.Fab")
+        (effects (font (size 1 1) (thickness 0.15)) (justify mirror))
+    )

Commit message: Polaroid board: match ordered parts; add JLC assembly files
- Values now name the parts ordered: C1 0.75pF, R1 240k, U1
  OPA365AIDBVR, F1 0.5A PPTC.
- R2 91k -> 100k (JLC basic part). The ADC divider ratio changes from
  0.622 to 0.600, so the max input is 3.15 V at 5.25 V. The firmware only
  uses relative thresholds.
- production_jlc/: BOM with LCSC numbers and CPL (bottom-side
  assembly). The rotations were checked against JLC's footprint for
  every part.

Co-Authored-By: Claude Opus 5.5 <noreply@anthropic.com>
Parts:
- C1: value (0.7pF) -> 0.75pF
- F1: value 0.5A -> 0.5A PPTC
- R1: value (240k) -> 240k
- R2: value 91k -> 100k
- U1: value OPA365xxDBV -> OPA365AIDBVR
Changed lines of the file:
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@@
         (effects (font (size 1 1) (thickness 0.15)) (justify mirror))
     )
-    (fp_text value "(0.7pF)" (at 0 -1.43) (layer "B.Fab")
+    (fp_text value "0.75pF" (at 0 -1.43) (layer "B.Fab")
         (effects (font (size 1 1) (thickness 0.15)) (justify mirror))
     )
@@
         (effects (font (size 1 1) (thickness 0.15)) (justify mirror))
     )
-    (fp_text value "(240k)" (at 0 -1.43) (layer "B.Fab")
+    (fp_text value "240k" (at 0 -1.43) (layer "B.Fab")
         (effects (font (size 1 1) (thickness 0.15)) (justify mirror))
     )
@@
         (effects (font (size 1 1) (thickness 0.15)) (justify mirror))
     )
-    (fp_text value "0.5A" (at 0 -1.82 90) (layer "B.Fab")
+    (fp_text value "0.5A PPTC" (at 0 -1.82 90) (layer "B.Fab")
         (effects (font (size 1 1) (thickness 0.15)) (justify mirror))
     )
@@
         (effects (font (size 1 1) (thickness 0.15)) (justify mirror))
     )
-    (fp_text value "91k" (at 0 -1.65) (layer "B.Fab")
+    (fp_text value "100k" (at 0 -1.65) (layer "B.Fab")
         (effects (font (size 1 1) (thickness 0.15)) (justify mirror))
     )
@@
         (effects (font (size 1 1) (thickness 0.15)) (justify mirror))
     )
-    (fp_text value "OPA365xxDBV" (at 0 -2.4) (layer "B.Fab")
-        (effects (font (size 1 1) (thickness 0.15)) (justify mirror))
-    )
+    (fp_text value "OPA365AIDBVR" (at 0 -2.4) (layer "B.Fab")
+        (effects (font (size 1 1) (thickness 0.15)) (justify mirror))
+    )
