File: pcb/pcb_for_Polaroid/ShutterCal_Polaroid/ShutterCal_Polaroid.kicad_sch (KiCad schematic)
At the start: 34 parts, among them J1 Conn_Coaxial, J2 Conn_01x04_Socket, J3 USB_C_Receptacle_USB2.0, J4 Conn_01x04_Socket, J5 Conn_01x04_Socket, J6 Conn_01x04_Shielded, J7 Conn_01x02_Socket, J9 Conn_01x04_Shielded, U1 OPA365xxDBV, U2 STM32G030F6Px, U3 CH340N, U4 AMS1117-3.3

Commit message: Polaroid board: fix R4/R5 reference divider and USB-C CC resistors
- R4/R5: the PCB routes R4 from GND to U1+ and R5 from U1+ to +5V, but
  the schematic had them the other way round (and the PCB footprints
  linked to deleted symbols, so parity matched by reference only). With
  the schematic values as routed, U1+ sat at ~4.9 V and the photodiode
  amp was saturated. The schematic now matches the routed copper: R4
  (6.8k) is on the GND side and R5 (330k) on the +5V side, giving
  ~0.10 V at U1+, which is what the firmware's dark threshold expects.
  The PCB footprints are relinked to the current symbols. Copper is
  unchanged.
- R6/R7 (USB-C CC1/CC2 pull-downs): 1k / not fitted -> 5.1k / 5.1k, as
  the Type-C spec requires for a sink, so C-to-C cables work in both
  plug orientations.

DRC: 0 unconnected, all 4 R4/R5 net conflicts gone; the remaining
warnings are unchanged.

Co-Authored-By: Claude Opus 5.5 <noreply@anthropic.com>
Parts:
- R4: value 330k -> 6.8k
- R5: value 6.8k -> 330k
- R6: value 1k -> 5.1k
- R7: value (1k)DNF -> 5.1k
Connections:
- net +5V: now also R5.2; no longer R4.2
- net GND: now also R4.1; no longer R5.1
- net at C2.1, TP1.1, U1.3 (+): now also R4.2, R5.1; no longer R4.1, R5.2
Other:
- moved on the sheet: R4, R5
Changed lines of the file:
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@@
+    )
+  )
+  (symbol (lib_id "Device:R") (at 49.53 57.15 180) (unit 1)
+    (in_bom yes) (on_board yes) (dnp no) (fields_autoplaced)
+    (property "Reference" "R5" (at 51.435 55.88 0)
+      (effects (font (size 1.27 1.27)) (justify right))
+    )
+    (property "Value" "330k" (at 51.435 58.42 0)
+      (effects (font (size 1.27 1.27)) (justify right))
+    )
+    (property "Footprint" "Resistor_SMD:R_0603_1608Metric" (at 51.308 57.15 90)
+      (effects (font (size 1.27 1.27)) hide)
+    )
+    (property "Datasheet" "~" (at 49.53 57.15 0)
+      (effects (font (size 1.27 1.27)) hide)
+    )
+    (pin "1")
+    (pin "2")
+    (instances
+      (project "ShutterCal_Polaroid"
+        (path "/67a01e2a-c6cc-4455-a1e5-78bdca908ff0"
+          (reference "R5") (unit 1)
+        )
+      )
+    )
+  )
+  (symbol (lib_id "Regulator_Linear:AMS1117-3.3") (at 243.84 95.885 0) (unit 1)
+    (in_bom yes) (on_board yes) (dnp no) (fields_autoplaced)
+    (property "Reference" "U4" (at 243.84 89.535 0)
+      (effects (font (size 1.27 1.27)))
+    )
+    (property "Value" "AMS1117-3.3" (at 243.84 92.075 0)
+      (effects (font (size 1.27 1.27)))
+    )
+    (property "Footprint" "Package_TO_SOT_SMD:SOT-223-3_TabPin2" (at 243.84 90.805 0)
+      (effects (font (size 1.27 1.27)) hide)
+    )
+    (property "Datasheet" "http://www.advanced-monolithic.com/pdf/ds1117.pdf" (at 246.38 102.235 0)
+      (effects (font (size 1.27 1.27)) hide)
+    )
+    (pin "1")
+    (pin "2")
+    (pin "3")
+    (instances
+      (project "ShutterCal_Polaroid"
+        (path "/67a01e2a-c6cc-4455-a1e5-78bdca908ff0"
+          (reference "U4") (unit 1)
+        )
+      )
     )
   )
   (symbol (lib_id "Device:R") (at 49.53 66.04 180) (unit 1)
     (in_bom yes) (on_board yes) (dnp no) (fields_autoplaced)
-    (property "Reference" "R5" (at 51.435 64.77 0)
+    (property "Reference" "R4" (at 51.435 64.77 0)
       (effects (font (size 1.27 1.27)) (justify right))
     )
@@
     )
     (property "Datasheet" "~" (at 49.53 66.04 0)
-      (effects (font (size 1.27 1.27)) hide)
-    )
-    (pin "1")
-    (pin "2")
-    (instances
-      (project "ShutterCal_Polaroid"
-        (path "/67a01e2a-c6cc-4455-a1e5-78bdca908ff0"
-          (reference "R5") (unit 1)
-        )
-      )
-    )
-  )
-  (symbol (lib_id "Regulator_Linear:AMS1117-3.3") (at 243.84 95.885 0) (unit 1)
-    (in_bom yes) (on_board yes) (dnp no) (fields_autoplaced)
-    (property "Reference" "U4" (at 243.84 89.535 0)
-      (effects (font (size 1.27 1.27)))
-    )
-    (property "Value" "AMS1117-3.3" (at 243.84 92.075 0)
-      (effects (font (size 1.27 1.27)))
-    )
-    (property "Footprint" "Package_TO_SOT_SMD:SOT-223-3_TabPin2" (at 243.84 90.805 0)
-      (effects (font (size 1.27 1.27)) hide)
-    )
-    (property "Datasheet" "http://www.advanced-monolithic.com/pdf/ds1117.pdf" (at 246.38 102.235 0)
-      (effects (font (size 1.27 1.27)) hide)
-    )
-    (pin "1")
-    (pin "2")
-    (pin "3")
-    (instances
-      (project "ShutterCal_Polaroid"
-        (path "/67a01e2a-c6cc-4455-a1e5-78bdca908ff0"
-          (reference "U4") (unit 1)
-        )
-      )
-    )
-  )
-  (symbol (lib_id "Device:R") (at 49.53 57.15 180) (unit 1)
-    (in_bom yes) (on_board yes) (dnp no) (fields_autoplaced)
-    (property "Reference" "R4" (at 51.435 55.88 0)
-      (effects (font (size 1.27 1.27)) (justify right))
-    )
-    (property "Value" "330k" (at 51.435 58.42 0)
-      (effects (font (size 1.27 1.27)) (justify right))
-    )
-    (property "Footprint" "Resistor_SMD:R_0603_1608Metric" (at 51.308 57.15 90)
-      (effects (font (size 1.27 1.27)) hide)
-    )
-    (property "Datasheet" "~" (at 49.53 57.15 0)
       (effects (font (size 1.27 1.27)) hide)
     )
@@
       (effects (font (size 1.27 1.27)))
     )
-    (property "Value" "(1k)DNF" (at 60.96 107.95 90)
+    (property "Value" "5.1k" (at 60.96 107.95 90)
       (effects (font (size 1.27 1.27)))
     )
@@
       (effects (font (size 1.27 1.27)))
     )
-    (property "Value" "1k" (at 53.34 104.14 90)
-      (effects (font (size 1.27 1.27)))
-    )
+    (property "Value" "5.1k" (at 53.34 104.14 90)
+      (effects (font (size 1.27 1.27)))
+    )

Commit message: Polaroid board: match ordered parts; add JLC assembly files
- Values now name the parts ordered: C1 0.75pF, R1 240k, U1
  OPA365AIDBVR, F1 0.5A PPTC.
- R2 91k -> 100k (JLC basic part). The ADC divider ratio changes from
  0.622 to 0.600, so the max input is 3.15 V at 5.25 V. The firmware only
  uses relative thresholds.
- production_jlc/: BOM with LCSC numbers and CPL (bottom-side
  assembly). The rotations were checked against JLC's footprint for
  every part.

Co-Authored-By: Claude Opus 5.5 <noreply@anthropic.com>
Parts:
- C1: value (0.7pF) -> 0.75pF
- F1: value 0.5A -> 0.5A PPTC
- R1: value (240k) -> 240k
- R2: value 91k -> 100k
- U1: value OPA365xxDBV -> OPA365AIDBVR
Changed lines of the file:
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@@
       (effects (font (size 1.27 1.27)))
     )
-    (property "Value" "OPA365xxDBV" (at 85.09 49.9109 0)
+    (property "Value" "OPA365AIDBVR" (at 85.09 49.9109 0)
       (effects (font (size 1.27 1.27)))
     )
@@
       (effects (font (size 1.27 1.27)))
     )
-    (property "Value" "(0.7pF)" (at 78.105 20.32 90)
+    (property "Value" "0.75pF" (at 78.105 20.32 90)
       (effects (font (size 1.27 1.27)))
     )
@@
       (effects (font (size 1.27 1.27)))
     )
-    (property "Value" "(240k)" (at 77.47 31.75 90)
+    (property "Value" "240k" (at 77.47 31.75 90)
       (effects (font (size 1.27 1.27)))
     )
@@
       (effects (font (size 1.27 1.27)) (justify left))
     )
-    (property "Value" "91k" (at 120.015 38.1 0)
+    (property "Value" "100k" (at 120.015 38.1 0)
       (effects (font (size 1.27 1.27)) (justify left))
     )
@@
       (effects (font (size 1.27 1.27)))
     )
-    (property "Value" "0.5A" (at 53.975 91.44 90)
-      (effects (font (size 1.27 1.27)))
-    )
+    (property "Value" "0.5A PPTC" (at 53.975 91.44 90)
+      (effects (font (size 1.27 1.27)))
+    )
